File: PCB/genius.kicad_pcb (KiCad board)
At the start: 2 copper layers, 71.1 x 78.7 mm, 20 parts, among them J1 PICKIT3_CONN, SW1 SW_Push, SW2 SW_Push, SW3 SW_Push, SW4 SW_Push, SW5 SW_Push, U1 L7805, U2 PIC16(L)F628A-I/P

Commit message: Rev. PCB
Parts:
- moved D2 3.00 mm to (80.8, 124.5)
- moved SW2 2.54 mm to (78.7, 132.1)
Routing:
- net Net-(SW2-Pad2): track 45.8 -> 43.9 mm
- net GND: track 213.3 -> 215.0 mm
- net Net-(D2-Pad2): track 7.62 -> 8.86 mm
